Commit message: Aggiunta ostacoli (non rileva le collisioni)

File: tm5_900/description/desc_tm900/urdf/tm5_900.urdf.xacro (robot description, xacro)
@@ -82,5 +82,5 @@
         </material>
       </visual>
-      <collision>
+      <collision name="base_link_collision">
         <geometry>
           <mesh filename="$(find tm5_900)/description/desc_tm900/meshes/tm5_900/collision/tm5_base_c.stl" />
@@ -113,5 +113,5 @@
         </material>
       </visual>
-      <collision>
+      <collision name="shoulder_1_link_collision">
         <geometry>
           <mesh filename="$(find tm5_900)/description/desc_tm900/meshes/tm5_900/collision/tm_400w_01_c.stl" />
@@ -144,5 +144,5 @@
         </material>
       </visual>
-      <collision>
+      <collision name="arm_1_link_collision">
         <geometry>
           <mesh filename="$(find tm5_900)/description/desc_tm900/meshes/tm5_900/collision/tm5_900_arm1_c.stl" />
@@ -175,5 +175,5 @@
         </material>
       </visual>
-      <collision>
+      <collision name="arm_2_link_collision">
         <geometry>
           <mesh filename="$(find tm5_900)/description/desc_tm900/meshes/tm5_900/collision/tm5_900_arm2_c.stl" />
@@ -206,5 +206,5 @@
         </material>
       </visual>
-      <collision>
+      <collision name="wrist_1_link_collision">
         <geometry>
           <mesh filename="$(find tm5_900)/description/desc_tm900/meshes/tm5_900/collision/tm_100w_01_c.stl" />
@@ -237,5 +237,5 @@
         </material>
       </visual>
-      <collision>
+      <collision name="wrist_2_link_collision">
         <geometry>
           <mesh filename="$(find tm5_900)/description/desc_tm900/meshes/tm5_900/collision/tm_100w_02_c.stl" />
@@ -268,5 +268,5 @@
         </material>
       </visual>
-      <collision>
+      <collision name="wrist_3_link_collision">
         <geometry>
           <mesh filename="$(find tm5_900)/description/desc_tm900/meshes/tm5_900/collision/tm_ee_c.stl" />
@@ -283,5 +283,5 @@
     </joint>
     <link name="flange_link">
-    </link>
+  </link>
     <!-- ROS base to TM 'base_link' Coordinates transform -->
     <link name="base" />

Commit message: Lettura ostacoli e inserimento manuale punto

File: tm5_900/description/desc_tm900/urdf/tm5_900.urdf.xacro (robot description, xacro)
@@ -82,5 +82,5 @@
         </material>
       </visual>
-      <collision name="base_link_collision">
+      <collision >
         <geometry>
           <mesh filename="$(find tm5_900)/description/desc_tm900/meshes/tm5_900/collision/tm5_base_c.stl" />
@@ -113,5 +113,5 @@
         </material>
       </visual>
-      <collision name="shoulder_1_link_collision">
+      <collision >
         <geometry>
           <mesh filename="$(find tm5_900)/description/desc_tm900/meshes/tm5_900/collision/tm_400w_01_c.stl" />
@@ -144,5 +144,5 @@
         </material>
       </visual>
-      <collision name="arm_1_link_collision">
+      <collision >
         <geometry>
           <mesh filename="$(find tm5_900)/description/desc_tm900/meshes/tm5_900/collision/tm5_900_arm1_c.stl" />
@@ -175,5 +175,5 @@
         </material>
       </visual>
-      <collision name="arm_2_link_collision">
+      <collision >
         <geometry>
           <mesh filename="$(find tm5_900)/description/desc_tm900/meshes/tm5_900/collision/tm5_900_arm2_c.stl" />
@@ -206,5 +206,5 @@
         </material>
       </visual>
-      <collision name="wrist_1_link_collision">
+      <collision >
         <geometry>
           <mesh filename="$(find tm5_900)/description/desc_tm900/meshes/tm5_900/collision/tm_100w_01_c.stl" />
@@ -237,5 +237,5 @@
         </material>
       </visual>
-      <collision name="wrist_2_link_collision">
+      <collision >
         <geometry>
           <mesh filename="$(find tm5_900)/description/desc_tm900/meshes/tm5_900/collision/tm_100w_02_c.stl" />
@@ -268,5 +268,5 @@
         </material>
       </visual>
-      <collision name="wrist_3_link_collision">
+      <collision >
         <geometry>
           <mesh filename="$(find tm5_900)/description/desc_tm900/meshes/tm5_900/collision/tm_ee_c.stl" />

File: tm5_900/description/desc_tm900/urdf/tm_bumper_config.xacro (robot description, xacro)
@@ -2,7 +2,4 @@
 <robot xmlns:xacro="http://www.ros.org/wiki/xacro">
 	<xacro:macro name="tm_bumper_ctr_sensor">
-		<!-- I need this for contact sensor, "bumper sensor"  -->
-		<!-- I create this file in order to detect self-collisions and collisions with the ground  -->
-		<!-- This helps me to detect if the end effect touch the ground so I can reset the environment -->
 		<gazebo reference="flange_link">
 			<!-- contact sensor -->
